File: schematic/sp400.sch (KiCad schematic (older format))
At the start: 45 parts, among them CN1 DB9_Female, CN2 Conn_01x13_Male, CN3 Conn_01x07_Male, CN4 Jack-DC, IC1 M5L8035LP, IC2 HD6805V, IC3 74LS04, IC4 74LS373, IC5 HN462732G, IC6 LB1257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

Commit message: started disassembling 6805
Parts:
- IC2: symbol MCU_Motorola_Fabio:6805 -> sp400-rescue:6805-MCU_Motorola_Fabio
Connections:
- net labels added: clk, d1, d2, d3, d7, xa, xb, xc, xd, ya, yb, yc, yd
- wire segments 75 -> 78
- no-connect marks 3 -> 4
Other:
- moved on the sheet: CN2, CN3, D2, D3, D4, D5, D6, IC3A
Changed lines of the file:
@@
-$EndComp
-$Comp
-L Connector:Conn_01x13_Male CN2
-U 1 1 613D146A
-P 7950 1550
-F 0 "CN2" H 8058 2331 50  0000 C CNN
-F 1 "Conn_01x13_Male" H 8058 2240 50  0000 C CNN
-F 2 "" H 7950 1550 50  0001 C CNN
-F 3 "~" H 7950 1550 50  0001 C CNN
-	1    7950 1550
-	1    0    0    -1
 $EndComp
 $Comp
 L Connector:Conn_01x07_Male CN3
 U 1 1 613D5070
-P 800 1250
-F 0 "CN3" H 908 1731 50  0000 C CNN
-F 1 "Conn_01x07_Male" H 908 1640 50  0000 C CNN
-F 2 "" H 800 1250 50  0001 C CNN
-F 3 "~" H 800 1250 50  0001 C CNN
-	1    800  1250
-	1    0    0    -1
+P 12700 8450
+F 0 "CN3" H 12808 8931 50  0000 C CNN
+F 1 "Conn_01x07_Male" H 12808 8840 50  0000 C CNN
+F 2 "" H 12700 8450 50  0001 C CNN
+F 3 "~" H 12700 8450 50  0001 C CNN
+	1    12700 8450
+	-1   0    0    -1
 $EndComp
 $Comp
@@
 L Device:D D2
 U 1 1 613EA2BE
-P 14150 5400
-F 0 "D2" H 14200 5300 50  0000 R CNN
-F 1 "D" H 14200 5500 50  0000 R CNN
-F 2 "" H 14150 5400 50  0001 C CNN
-F 3 "~" H 14150 5400 50  0001 C CNN
-	1    14150 5400
+P 13950 6800
+F 0 "D2" H 14000 6700 50  0000 R CNN
+F 1 "D" H 14000 6900 50  0000 R CNN
+F 2 "" H 13950 6800 50  0001 C CNN
+F 3 "~" H 13950 6800 50  0001 C CNN
+	1    13950 6800
 	1    0    0    -1
 $EndComp
@@
 L Device:D D4
 U 1 1 613EAC97
-P 14150 6000
-F 0 "D4" H 14100 5750 50  0000 L CNN
-F 1 "D" H 14150 5850 50  0000 L CNN
-F 2 "" H 14150 6000 50  0001 C CNN
-F 3 "~" H 14150 6000 50  0001 C CNN
-	1    14150 6000
+P 13950 7400
+F 0 "D4" H 13900 7150 50  0000 L CNN
+F 1 "D" H 13950 7250 50  0000 L CNN
+F 2 "" H 13950 7400 50  0001 C CNN
+F 3 "~" H 13950 7400 50  0001 C CNN
+	1    13950 7400
 	-1   0    0    1
 $EndComp
@@
 L Device:D D6
 U 1 1 613EB583
-P 13950 5650
-F 0 "D6" H 13950 5867 50  0000 C CNN
-F 1 "D" H 13950 5776 50  0000 C CNN
-F 2 "" H 13950 5650 50  0001 C CNN
-F 3 "~" H 13950 5650 50  0001 C CNN
-	1    13950 5650
+P 13750 7050
+F 0 "D6" H 13750 7267 50  0000 C CNN
+F 1 "D" H 13750 7176 50  0000 C CNN
+F 2 "" H 13750 7050 50  0001 C CNN
+F 3 "~" H 13750 7050 50  0001 C CNN
+	1    13750 7050
 	0    1    1    0
 $EndComp
@@
 $EndComp
 $Comp
-L MCU_Motorola_Fabio:6805 IC2
+L sp400-rescue:6805-MCU_Motorola_Fabio IC2
 U 1 1 613F663D
 P 11200 5500
@@
 L 74xx:74LS04 IC3
 U 1 1 6140ED41
-P 4400 6350
-F 0 "IC3" H 4400 6667 50  0000 C CNN
-F 1 "74LS04" H 4400 6576 50  0000 C CNN
-F 2 "" H 4400 6350 50  0001 C CNN
-F 3 "http://www.ti.com/lit/gpn/sn74LS04" H 4400 6350 50  0001 C CNN
-	1    4400 6350
+P 11900 8150
+F 0 "IC3" H 11900 8467 50  0000 C CNN
+F 1 "74LS04" H 11900 8376 50  0000 C CNN
+F 2 "" H 11900 8150 50  0001 C CNN
+F 3 "http://www.ti.com/lit/gpn/sn74LS04" H 11900 8150 50  0001 C CNN
+	1    11900 8150
 	1    0    0    -1
 $EndComp
@@
 Text Label 10750 6650 2    50   ~ 0
 d6
-Text Label 6600 5300 2    50   ~ 0
-d6
 Text Label 10750 6550 2    50   ~ 0
-d5
-Text Label 6600 5200 2    50   ~ 0
 d5
 Text Label 10750 6450 2    50   ~ 0
 d4
-Text Label 6600 5100 2    50   ~ 0
-d4
 Text Label 10750 6050 2    50   ~ 0
-d0
-Text Label 6600 4700 2    50   ~ 0
 d0
 Wire Wire Line
@@
 L Device:D D5
 U 1 1 61755749
-P 13750 6000
-F 0 "D5" H 13750 6217 50  0000 C CNN
-F 1 "D" H 13750 6126 50  0000 C CNN
-F 2 "" H 13750 6000 50  0001 C CNN
-F 3 "~" H 13750 6000 50  0001 C CNN
-	1    13750 6000
-	1    0    0    -1
-$EndComp
-Wire Wire Line
-	14000 6000 13950 6000
+P 13550 7400
+F 0 "D5" H 13550 7617 50  0000 C CNN
+F 1 "D" H 13550 7526 50  0000 C CNN
+F 2 "" H 13550 7400 50  0001 C CNN
+F 3 "~" H 13550 7400 50  0001 C CNN
+	1    13550 7400
+	1    0    0    -1
+$EndComp
+Wire Wire Line
+	13800 7400 13750 7400
 $Comp
 L Device:D D3
 U 1 1 617630AF
-P 13750 5400
-F 0 "D3" H 13800 5500 50  0000 R CNN
-F 1 "D" H 13750 5300 50  0000 R CNN
-F 2 "" H 13750 5400 50  0001 C CNN
-F 3 "~" H 13750 5400 50  0001 C CNN
-	1    13750 5400
+P 13550 6800
+F 0 "D3" H 13600 6900 50  0000 R CNN
+F 1 "D" H 13550 6700 50  0000 R CNN
+F 2 "" H 13550 6800 50  0001 C CNN
+F 3 "~" H 13550 6800 50  0001 C CNN
+	1    13550 6800
 	-1   0    0    1
 $EndComp
 Wire Wire Line
-	14000 5400 13950 5400
-Wire Wire Line
-	14300 6000 14350 6000
-Wire Wire Line
-	14350 6000 14350 5400
-Wire Wire Line
-	14350 5400 14300 5400
-Wire Wire Line
-	13950 6000 13950 5800
-Connection ~ 13950 6000
-Wire Wire Line
-	13950 6000 13900 6000
-Wire Wire Line
-	13950 5500 13950 5400
-Connection ~ 13950 5400
-Wire Wire Line
-	13950 5400 13900 5400
+	13800 6800 13750 6800
+Wire Wire Line
+	14100 7400 14150 7400
+Wire Wire Line
+	14150 7400 14150 6800
+Wire Wire Line
+	14150 6800 14100 6800
+Wire Wire Line
+	13750 7400 13750 7200
+Connection ~ 13750 7400
+Wire Wire Line
+	13750 7400 13700 7400
+Wire Wire Line
+	13750 6900 13750 6800
+Connection ~ 13750 6800
+Wire Wire Line
+	13750 6800 13700 6800
 Wire Wire Line
 	11650 4850 11950 4850
@@
 	12450 5050 12450 4950
 Connection ~ 12450 4950
+Text Label 10750 6150 2    50   ~ 0
+d1
+Text Label 10750 6250 2    50   ~ 0
+d2
+Text Label 10750 6350 2    50   ~ 0
+d3
+Text Label 10750 6750 2    50   ~ 0
+d7
+Text Label 6600 5300 2    50   ~ 0
+d6
+Text Label 6600 5200 2    50   ~ 0
+d5
+Text Label 6600 5100 2    50   ~ 0
+d4
+Text Label 6600 4700 2    50   ~ 0
+d0
+Text Label 6600 4800 2    50   ~ 0
+d1
+Text Label 6600 4900 2    50   ~ 0
+d2
+Text Label 6600 5000 2    50   ~ 0
+d3
+Text Label 6600 5400 2    50   ~ 0
+d7
+Text Label 10100 4950 0    50   ~ 0
+clk
+Text Label 8000 6700 0    50   ~ 0
+clk
+NoConn ~ 8000 6900
+Text Label 14000 5450 2    50   ~ 0
+xd
+Text Label 14000 5550 2    50   ~ 0
+xc
+Text Label 14000 5650 2    50   ~ 0
+xb
+Text Label 14000 5750 2    50   ~ 0
+xa
+$Comp
+L Connector:Conn_01x13_Male CN2
+U 1 1 613D146A
+P 14200 5850
+F 0 "CN2" H 14308 6631 50  0000 C CNN
+F 1 "Conn_01x13_Male" H 14308 6540 50  0000 C CNN
+F 2 "" H 14200 5850 50  0001 C CNN
+F 3 "~" H 14200 5850 50  0001 C CNN
+	1    14200 5850
+	-1   0    0    -1
+$EndComp
+Text Label 14000 5950 2    50   ~ 0
+yd
+Text Label 14000 6050 2    50   ~ 0
+yc
+Text Label 14000 6150 2    50   ~ 0
+yb
+Text Label 14000 6250 2    50   ~ 0
+ya
+Text Label 13100 6150 0    50   ~ 0
+xd
+Text Label 13100 6050 0    50   ~ 0
+xc
+Text Label 13100 5950 0    50   ~ 0
+xb
+Text Label 13100 5850 0    50   ~ 0
+xa
+Text Label 13100 5750 0    50   ~ 0
+yd
+Text Label 13100 5650 0    50   ~ 0
+yc
+Text Label 13100 5550 0    50   ~ 0
+yb
+Text Label 13100 5450 0    50   ~ 0
+ya
+$Comp
+L power:GND #PWR?
+U 1 1 622724C5
+P 12450 8850
+F 0 "#PWR?" H 12450 8600 50  0001 C CNN
+F 1 "GND" H 12455 8677 50  0000 C CNN
+F 2 "" H 12450 8850 50  0001 C CNN
+F 3 "" H 12450 8850 50  0001 C CNN
+	1    12450 8850
+	-1   0    0    -1
+$EndComp
+Wire Wire Line
+	12500 8750 12450 8750
+Wire Wire Line
+	12450 8750 12450 8850
+Wire Wire Line
+	12200 8150 12500 8150
+Text Label 11600 8150 2    50   ~ 0
+busy
 $EndSCHEMATC

Commit message: panel connector added
Parts:
- removed CN1: DB9_Female, symbol Connector:DB9_Female
- added CN6: Conn_01x07_Female, symbol Connector:Conn_01x07_Female
- added CNEDGE: Conn_01x13_Female, symbol Connector:Conn_01x13_Female
- added D?: green, symbol Device:LED
- added D?: red, symbol Device:LED
- added J?: DB9_Male, symbol Connector:DB9_Male
- added SW?: CHANGE COLOR, symbol Switch:SW_Push
- added SW?: CHANGE PEN, symbol Switch:SW_Push
- added SW?: LINE FEED, symbol Switch:SW_Push
- IC2: symbol sp400-rescue:6805-MCU_Motorola_Fabio -> MCU_Motorola_Fabio:6805
Connections:
- net labels added: changeColor, changePen, data, lineFeed, p25
- net labels removed: clk, d1, d2, d3, d7, xa, xb, xc, xd, ya, yb, yc, yd
- wire segments 78 -> 123
- no-connect marks 4 -> 9
Other:
- note added: "black"
- note added: "blue"
- note added: "brown"
- note added: "gray"
- note added: "green"
- note added: "lightblue"
- note added: "lightgreen"
- note added: "orange"
- note added: "pink"
- note added: "purple"
- note added: "red"
- note added: "white"
- note added: "yellow"
- moved on the sheet: C10, C4, CN2, CN3, D2, D3, D4, D5, D6, IC3A, IC3E, IC3F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
